File: kicad/modules/hellen1-motor-driver/hellen1-motor-driver.kicad_sch (KiCad schematic)
At the start: 17 parts, among them M821 Module-motor-driver-0.1

Commit message: https://github.com/rusefi/uaefi121/issues/22
Other:
- title: MCZ33810 module -> Motor-driver module
