File: kicad/modules/hellen1-vr-discrete/hellen1-vr-discrete.kicad_pcb (KiCad board)
At the start: 4 copper layers, 15.2 x 9.8 mm, 47 parts, among them M750 Module-vr-discrete-0.2, U751 SRV05-4-P-T7, U752 74AHC1G02, U753 MCP6004, U754 MAX9142, U755 NC7SB3157P6X, U756 NC7SB3157P6X, U757 74AHC1G02

Commit message: vr-discrete 0.5 #375
Parts:
- added R770: DNP, Resistor_SMD:R_0402_1005Metric, F.Cu at (81.9, 90.4)
- M750: value Module-vr-discrete-0.2 -> Module-vr-discrete-0.5; footprint hellen-one-vr-discrete-0.2:vr-discrete -> hellen-one-vr-discrete-0.5:vr-discrete
- moved D751 0.37 mm to (79.6, 89.3)
- moved C765 0.06 mm to (82.3, 88.7)
Routing:
- net Net-(U751-IO2): track 6.36 -> 15.4 mm, vias 1 -> 2
- net output: track 21.3 -> 19.0 mm
- net GND: track 1.97 -> 2.72 mm, vias 19 -> 18
- net +5V: track 52.7 -> 52.2 mm
