File: kicad/modules/hellen1-mcz33810/hellen1-mcz33810.kicad_sch (KiCad schematic)
At the start: 32 parts, among them M801 Module-mcz33810-0.1, U9 MCZ33810EK

Commit message: #382
Other:
- note added: "Remove R806, R808, R810, R812, Q801-Q804, C806-C809 and install 0 Ohm R814-R817 for use with smart coils"
Changed lines of the file:
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@@
     (stroke (width 0) (type default))
+  )
+  (text "Remove R806, R808, R810, R812, Q801-Q804, C806-C809\nand install 0 Ohm R814-R817 for use with smart coils"
+    (at 215.9 40.64 0)
+    (effects (font (size 1.27 1.27)) (justify left bottom))
   )
   (label "IGN1" (at 83.82 27.94 0) (fields_autoplaced)
